Commit message: Seperate the arm using macro

File: kumara_description/urdf/kumara.xacro (robot description, xacro)
@@ -1,8 +1,8 @@
 <?xml version="1.0"?>
 <robot name="Kumara" xmlns:xacro="http://www.ros.org/wiki/xacro">
-    <xacro:include filename="$(find kumara_description)/urdf/materials.xacro" />
     <xacro:include filename="$(find kumara_description)/urdf/kumara_properties.xacro" />
     <xacro:include filename="$(find kumara_description)/urdf/kumara.gazebo" />
-    <!-- <link name="base_footprint"/> -->
+    <xacro:include filename="$(find kumara_description)/urdf/kumara_arm.xacro" />
+    <xacro:kumaraRA parent = "chassis"/>
     <link name="base_footprint"/>
     <link name="chassis">
@@ -22,81 +22,4 @@
                 <mesh filename="package://kumara_description/meshes/base/kumaraBaseV2.STL" scale="1 1 1"/>
             </geometry>
-            <!-- <material name="orange"/> -->
-        </visual>
-    </link>
-    <link name="arm_base">
-		<inertial>
-			<mass value = "1"/>
-			<inertia ixx = "0.26" iyy = "0.26" izz = "0.01" ixy = "0" ixz = "0" iyz = "0"/>
-		</inertial>
-        <visual>
-            <geometry>
-                <mesh filename="package://kumara_description/meshes/arm/base_link.STL" scale="1 1 1"/>
-            </geometry>
-        </visual>
-    </link>
-    <link name="link_1">
-		<inertial>
-            <origin rpy="${PId2} 0 0" xyz = "0 0 ${L1}"/>
-			<mass value = "1"/>
-			<inertia ixx = "0.26" iyy = "0.26" izz = "0.01" ixy = "0" ixz = "0" iyz = "0"/>
-		</inertial>
-        <visual>
-            <origin rpy="${PId2} 0 0" xyz = "0 0 ${L1}"/>
-            <geometry>
-                <mesh filename="package://kumara_description/meshes/arm/link_1.STL" scale="1 1 1"/>
-            </geometry>
-        </visual>
-    </link>
-    <link name="link_2">
-		<inertial>
-            <origin rpy="-${PId2} 0 ${PId2}"/>
-			<mass value = "1"/>
-			<inertia ixx = "0.26" iyy = "0.26" izz = "0.01" ixy = "0" ixz = "0" iyz = "0"/>
-		</inertial>
-        <visual>
-            <origin rpy="-${PId2} 0 ${PId2}"/>
-            <geometry>
-                <mesh filename="package://kumara_description/meshes/arm/link_2.STL" scale="1 1 1"/>
-            </geometry>
-        </visual>
-    </link>
-    <link name="link_3">
-		<inertial>
-            <origin rpy="-${PId2} 0 -${PId2}" xyz = "0 0 ${L2}"/>
-			<mass value = "1"/>
-			<inertia ixx = "0.26" iyy = "0.26" izz = "0.01" ixy = "0" ixz = "0" iyz = "0"/>
-		</inertial>
-        <visual>
-            <origin rpy="-${PId2} 0 -${PId2}" xyz = "0 0 ${L2}"/>
-            <geometry>
-                <mesh filename="package://kumara_description/meshes/arm/link_3.STL" scale="1 1 1"/>
-            </geometry>
-        </visual>
-    </link>
-    <link name="link_4">
-		<inertial>
-            <origin rpy="${PId2} 0 ${PId2}"/>
-			<mass value = "1"/>
-			<inertia ixx = "0.26" iyy = "0.26" izz = "0.01" ixy = "0" ixz = "0" iyz = "0"/>
-		</inertial>
-        <visual>
-            <origin rpy="${PId2} 0 ${PId2}"/>
-            <geometry>
-                <mesh filename="package://kumara_description/meshes/arm/link_4.STL" scale="1 1 1"/>
-            </geometry>
-        </visual>
-    </link>
-    <link name="link_5">
-		<inertial>
-            <origin xyz="0 0 ${L3}"/>
-			<mass value = "1"/>
-			<inertia ixx = "0.26" iyy = "0.26" izz = "0.01" ixy = "0" ixz = "0" iyz = "0"/>
-		</inertial>
-        <visual>
-            <origin xyz="0 0 ${L3}"/>
-            <geometry>
-                <mesh filename="package://kumara_description/meshes/arm/link_5.STL" scale="1 1 1"/>
-            </geometry>
         </visual>
     </link>
@@ -108,44 +31,3 @@
         <limit effort = "50" velocity = "10"/>
     </joint>
-    <joint name="chassis_to_arm_base" type="revolute">
-        <parent link="chassis"/>
-        <child link="arm_base"/>
-        <origin xyz="0.17717 -0.0752 0.97939" rpy = "${PId2} -${PId2} 0"/>
-        <axis xyz = "0 0 1"/>
-        <limit lower = "-${PI}" upper = "${PI}" effort = "50" velocity = "10"/>
-    </joint>
-    <joint name="arm_base_to_link_1" type="revolute">
-        <parent link="arm_base"/>
-        <child link="link_1"/>
-        <axis xyz = "0 0 1"/>
-        <limit lower = "-${PI}" upper = "${PI}" effort = "50" velocity = "10"/>
-    </joint>
-    <joint name="link_1_to_link_2" type="revolute">
-        <parent link="link_1"/>
-        <child link="link_2"/>
-        <axis xyz = "0 0 1"/>
-        <origin rpy="${PId2} 0 0" xyz = "0 0 0.13764"/>
-        <limit lower = "-${PI}" upper = "${PI}" effort = "50" velocity = "10"/>
-    </joint>
-    <joint name="link_2_to_link_3" type="revolute">
-        <parent link="link_2"/>
-        <child link="link_3"/>
-        <axis xyz = "0 0 1"/>
-        <origin rpy="-${PId2} 0 ${PId2}"/>
-        <limit lower = "-${PI}" upper = "${PI}" effort = "50" velocity = "10"/>
-    </joint>
-    <joint name="link_3_to_link_4" type="revolute">
-        <parent link="link_3"/>
-        <child link="link_4"/>
-        <axis xyz = "0 0 1"/>
-        <origin rpy="-${PId2} 0 -${PId2}" xyz = "0 0 0.27597"/>
-        <limit lower = "-${PI}" upper = "${PI}" effort = "50" velocity = "10"/>
-    </joint>
-    <joint name="link_4_to_link_5" type="revolute">
-        <parent link="link_4"/>
-        <child link="link_5"/>
-        <axis xyz = "0 0 1"/>
-        <origin rpy="${PId2} 0 ${PId2}"/>
-        <limit lower = "-${PI}" upper = "${PI}" effort = "50" velocity = "10"/>
-    </joint>
 </robot>

File: kumara_description/urdf/kumara_arm.xacro (robot description, xacro)
@@ -1,116 +1,124 @@
 <?xml version="1.0"?>
-<robot name="Kumara" xmlns:xacro="http://www.ros.org/wiki/xacro">
-    <xacro:include filename="$(find kumara_description)/urdf/materials.xacro" />
+<robot name="KumaraRA" xmlns:xacro="http://www.ros.org/wiki/xacro">
     <xacro:include filename="$(find kumara_description)/urdf/kumara_properties.xacro" />
     <xacro:include filename="$(find kumara_description)/urdf/kumara.gazebo" />
-    <link name="arm_base">
-		<inertial>
-			<mass value = "1"/>
-			<inertia ixx = "0.26" iyy = "0.26" izz = "0.01" ixy = "0" ixz = "0" iyz = "0"/>
-		</inertial>
-        <visual>
-            <geometry>
-                <mesh filename="package://kumara_description/meshes/arm/base_link.STL" scale="1 1 1"/>
-            </geometry>
-        </visual>
-    </link>
-    <link name="link_1">
-		<inertial>
-            <origin rpy="${PId2} 0 0" xyz = "0 0 ${L1}"/>
-			<mass value = "1"/>
-			<inertia ixx = "0.26" iyy = "0.26" izz = "0.01" ixy = "0" ixz = "0" iyz = "0"/>
-		</inertial>
-        <visual>
-            <origin rpy="${PId2} 0 0" xyz = "0 0 ${L1}"/>
-            <geometry>
-                <mesh filename="package://kumara_description/meshes/arm/link_1.STL" scale="1 1 1"/>
-            </geometry>
-        </visual>
-    </link>
-    <link name="link_2">
-		<inertial>
+    <xacro:macro name="kumaraRA" params="parent">
+        <link name="arm_base">
+            <inertial>
+                <mass value = "1"/>
+                <inertia ixx = "0.26" iyy = "0.26" izz = "0.01" ixy = "0" ixz = "0" iyz = "0"/>
+            </inertial>
+            <visual>
+                <geometry>
+                    <mesh filename="package://kumara_description/meshes/arm/base_link.STL" scale="1 1 1"/>
+                </geometry>
+            </visual>
+        </link>
+        <link name="link_1">
+            <inertial>
+                <origin rpy="${PId2} 0 0" xyz = "0 0 ${L1}"/>
+                <mass value = "1"/>
+                <inertia ixx = "0.26" iyy = "0.26" izz = "0.01" ixy = "0" ixz = "0" iyz = "0"/>
+            </inertial>
+            <visual>
+                <origin rpy="${PId2} 0 0" xyz = "0 0 ${L1}"/>
+                <geometry>
+                    <mesh filename="package://kumara_description/meshes/arm/link_1.STL" scale="1 1 1"/>
+                </geometry>
+            </visual>
+        </link>
+        <link name="link_2">
+            <inertial>
+                <origin rpy="-${PId2} 0 ${PId2}"/>
+                <mass value = "1"/>
+                <inertia ixx = "0.26" iyy = "0.26" izz = "0.01" ixy = "0" ixz = "0" iyz = "0"/>
+            </inertial>
+            <visual>
+                <origin rpy="-${PId2} 0 ${PId2}"/>
+                <geometry>
+                    <mesh filename="package://kumara_description/meshes/arm/link_2.STL" scale="1 1 1"/>
+                </geometry>
+            </visual>
+        </link>
+        <link name="link_3">
+            <inertial>
+                <origin rpy="-${PId2} 0 -${PId2}" xyz = "0 0 ${L2}"/>
+                <mass value = "1"/>
+                <inertia ixx = "0.26" iyy = "0.26" izz = "0.01" ixy = "0" ixz = "0" iyz = "0"/>
+            </inertial>
+            <visual>
+                <origin rpy="-${PId2} 0 -${PId2}" xyz = "0 0 ${L2}"/>
+                <geometry>
+                    <mesh filename="package://kumara_description/meshes/arm/link_3.STL" scale="1 1 1"/>
+                </geometry>
+            </visual>
+        </link>
+        <link name="link_4">
+            <inertial>
+                <origin rpy="${PId2} 0 ${PId2}"/>
+                <mass value = "1"/>
+                <inertia ixx = "0.26" iyy = "0.26" izz = "0.01" ixy = "0" ixz = "0" iyz = "0"/>
+            </inertial>
+            <visual>
+                <origin rpy="${PId2} 0 ${PId2}"/>
+                <geometry>
+                    <mesh filename="package://kumara_description/meshes/arm/link_4.STL" scale="1 1 1"/>
+                </geometry>
+            </visual>
+        </link>
+        <link name="link_5">
+            <inertial>
+                <origin xyz="0 0 ${L3}"/>
+                <mass value = "1"/>
+                <inertia ixx = "0.26" iyy = "0.26" izz = "0.01" ixy = "0" ixz = "0" iyz = "0"/>
+            </inertial>
+            <visual>
+                <origin xyz="0 0 ${L3}"/>
+                <geometry>
+                    <mesh filename="package://kumara_description/meshes/arm/link_5.STL" scale="1 1 1"/>
+                </geometry>
+            </visual>
+        </link>
+        <joint name="parent_to_arm_base" type="revolute">
+            <parent link="${parent}"/>
+            <child link="arm_base"/>
+            <axis xyz = "0 0 1"/>
+            <origin xyz="0.17717 -0.0752 0.97939" rpy = "${PId2} -${PId2} 0"/>
+            <limit lower = "-${PI}" upper = "${PI}" effort = "50" velocity = "10"/>
+        </joint>
+        <joint name="arm_base_to_link_1" type="revolute">
+            <parent link="arm_base"/>
+            <child link="link_1"/>
+            <axis xyz = "0 0 1"/>
+            <limit lower = "-${PI}" upper = "${PI}" effort = "50" velocity = "10"/>
+        </joint>
+        <joint name="link_1_to_link_2" type="revolute">
+            <parent link="link_1"/>
+            <child link="link_2"/>
+            <axis xyz = "0 0 1"/>
+            <origin rpy="${PId2} 0 0" xyz = "0 0 0.13764"/>
+            <limit lower = "-${PI}" upper = "${PI}" effort = "50" velocity = "10"/>
+        </joint>
+        <joint name="link_2_to_link_3" type="revolute">
+            <parent link="link_2"/>
+            <child link="link_3"/>
+            <axis xyz = "0 0 1"/>
             <origin rpy="-${PId2} 0 ${PId2}"/>
-			<mass value = "1"/>
-			<inertia ixx = "0.26" iyy = "0.26" izz = "0.01" ixy = "0" ixz = "0" iyz = "0"/>
-		</inertial>
-        <visual>
-            <origin rpy="-${PId2} 0 ${PId2}"/>
-            <geometry>
-                <mesh filename="package://kumara_description/meshes/arm/link_2.STL" scale="1 1 1"/>
-            </geometry>
-        </visual>
-    </link>
-    <link name="link_3">
-		<inertial>
-            <origin rpy="-${PId2} 0 -${PId2}" xyz = "0 0 ${L2}"/>
-			<mass value = "1"/>
-			<inertia ixx = "0.26" iyy = "0.26" izz = "0.01" ixy = "0" ixz = "0" iyz = "0"/>
-		</inertial>
-        <visual>
-            <origin rpy="-${PId2} 0 -${PId2}" xyz = "0 0 ${L2}"/>
-            <geometry>
-                <mesh filename="package://kumara_description/meshes/arm/link_3.STL" scale="1 1 1"/>
-            </geometry>
-        </visual>
-    </link>
-    <link name="link_4">
-		<inertial>
+            <limit lower = "-${PI}" upper = "${PI}" effort = "50" velocity = "10"/>
+        </joint>
+        <joint name="link_3_to_link_4" type="revolute">
+            <parent link="link_3"/>
+            <child link="link_4"/>
+            <axis xyz = "0 0 1"/>
+            <origin rpy="-${PId2} 0 -${PId2}" xyz = "0 0 0.27597"/>
+            <limit lower = "-${PI}" upper = "${PI}" effort = "50" velocity = "10"/>
+        </joint>
+        <joint name="link_4_to_link_5" type="revolute">
+            <parent link="link_4"/>
+            <child link="link_5"/>
+            <axis xyz = "0 0 1"/>
             <origin rpy="${PId2} 0 ${PId2}"/>
-			<mass value = "1"/>
-			<inertia ixx = "0.26" iyy = "0.26" izz = "0.01" ixy = "0" ixz = "0" iyz = "0"/>
-		</inertial>
-        <visual>
-            <origin rpy="${PId2} 0 ${PId2}"/>
-            <geometry>
-                <mesh filename="package://kumara_description/meshes/arm/link_4.STL" scale="1 1 1"/>
-            </geometry>
-        </visual>
-    </link>
-    <link name="link_5">
-		<inertial>
-            <origin xyz="0 0 ${L3}"/>
-			<mass value = "1"/>
-			<inertia ixx = "0.26" iyy = "0.26" izz = "0.01" ixy = "0" ixz = "0" iyz = "0"/>
-		</inertial>
-        <visual>
-            <origin xyz="0 0 ${L3}"/>
-            <geometry>
-                <mesh filename="package://kumara_description/meshes/arm/link_5.STL" scale="1 1 1"/>
-            </geometry>
-        </visual>
-    </link>
-    <joint name="arm_base_to_link_1" type="revolute">
-        <parent link="arm_base"/>
-        <child link="link_1"/>
-        <axis xyz = "0 0 1"/>
-        <limit lower = "-${PI}" upper = "${PI}" effort = "50" velocity = "10"/>
-    </joint>
-    <joint name="link_1_to_link_2" type="revolute">
-        <parent link="link_1"/>
-        <child link="link_2"/>
-        <axis xyz = "0 0 1"/>
-        <origin rpy="${PId2} 0 0" xyz = "0 0 0.13764"/>
-        <limit lower = "-${PI}" upper = "${PI}" effort = "50" velocity = "10"/>
-    </joint>
-    <joint name="link_2_to_link_3" type="revolute">
-        <parent link="link_2"/>
-        <child link="link_3"/>
-        <axis xyz = "0 0 1"/>
-        <origin rpy="-${PId2} 0 ${PId2}"/>
-        <limit lower = "-${PI}" upper = "${PI}" effort = "50" velocity = "10"/>
-    </joint>
-    <joint name="link_3_to_link_4" type="revolute">
-        <parent link="link_3"/>
-        <child link="link_4"/>
-        <axis xyz = "0 0 1"/>
-        <origin rpy="-${PId2} 0 -${PId2}" xyz = "0 0 0.27597"/>
-        <limit lower = "-${PI}" upper = "${PI}" effort = "50" velocity = "10"/>
-    </joint>
-    <joint name="link_4_to_link_5" type="revolute">
-        <parent link="link_4"/>
-        <child link="link_5"/>
-        <axis xyz = "0 0 1"/>
-        <origin rpy="${PId2} 0 ${PId2}"/>
-        <limit lower = "-${PI}" upper = "${PI}" effort = "50" velocity = "10"/>
-    </joint>
+            <limit lower = "-${PI}" upper = "${PI}" effort = "50" velocity = "10"/>
+        </joint>
+    </xacro:macro>
 </robot>

Commit message: add transmission and control

File: kumara_description/urdf/kumara.xacro (robot description, xacro)
@@ -1,6 +1,12 @@
 <?xml version="1.0"?>
 <robot name="Kumara" xmlns:xacro="http://www.ros.org/wiki/xacro">
+    <gazebo>
+        <plugin name="gazebo_ros_control" filename="libgazebo_ros_control.so">
+            <robotNamespace>/kumara</robotNamespace>
+        </plugin>
+    </gazebo>
     <xacro:include filename="$(find kumara_description)/urdf/kumara_properties.xacro" />
-    <xacro:include filename="$(find kumara_description)/urdf/kumara.gazebo" />
+    <xacro:include filename="$(find kumara_description)/urdf/kumara_base.gazebo" />
+    <!-- ARM -->
     <xacro:include filename="$(find kumara_description)/urdf/kumara_arm.xacro" />
     <xacro:kumaraRA parent = "chassis"/>
@@ -8,7 +14,7 @@
     <link name="chassis">
         <collision>
-			<origin xyz="0 0 ${-0.23/2}"/>
+			<origin xyz="0 0 -${0.23/2}"/>
 			<geometry>
-				<box size = "0.2 0.2 0.23"/>
+				<box size = "${BASE_LENGTH} ${BASE_WIDTH} ${BASE_HEIGHT}"/>
 			</geometry>
 		</collision>
@@ -27,5 +33,5 @@
         <parent link="base_footprint"/>
         <child link="chassis"/>
-        <origin xyz="0 0 0.23"/>
+        <origin xyz="0 0 ${BASE_HEIGHT}"/>
         <axis xyz = "0 1 0"/>
         <limit effort = "50" velocity = "10"/>

File: kumara_description/urdf/kumara_arm.xacro (robot description, xacro)
@@ -2,5 +2,5 @@
 <robot name="KumaraRA" xmlns:xacro="http://www.ros.org/wiki/xacro">
     <xacro:include filename="$(find kumara_description)/urdf/kumara_properties.xacro" />
-    <xacro:include filename="$(find kumara_description)/urdf/kumara.gazebo" />
+    <xacro:include filename="$(find kumara_description)/urdf/kumara_arm.gazebo" />
     <xacro:macro name="kumaraRA" params="parent">
         <link name="arm_base">
@@ -80,10 +80,11 @@
             </visual>
         </link>
-        <joint name="parent_to_arm_base" type="revolute">
+        <joint name="parent_to_arm_base" type="fixed">
             <parent link="${parent}"/>
             <child link="arm_base"/>
             <axis xyz = "0 0 1"/>
             <origin xyz="0.17717 -0.0752 0.97939" rpy = "${PId2} -${PId2} 0"/>
-            <limit lower = "-${PI}" upper = "${PI}" effort = "50" velocity = "10"/>
+            <dynamics damping="0.7"/>
+            <limit lower = "-${PI}" upper = "${PI}" effort = "40" velocity = "1000"/>
         </joint>
         <joint name="arm_base_to_link_1" type="revolute">
@@ -91,5 +92,6 @@
             <child link="link_1"/>
             <axis xyz = "0 0 1"/>
-            <limit lower = "-${PI}" upper = "${PI}" effort = "50" velocity = "10"/>
+            <dynamics damping="0.7"/>
+            <limit lower = "-${PI}" upper = "${PI}" effort = "40" velocity = "1000"/>
         </joint>
         <joint name="link_1_to_link_2" type="revolute">
@@ -98,5 +100,6 @@
             <axis xyz = "0 0 1"/>
             <origin rpy="${PId2} 0 0" xyz = "0 0 0.13764"/>
-            <limit lower = "-${PI}" upper = "${PI}" effort = "50" velocity = "10"/>
+            <dynamics damping="0.7"/>
+            <limit lower = "-${PI}" upper = "${PI}" effort = "40" velocity = "1000"/>
         </joint>
         <joint name="link_2_to_link_3" type="revolute">
@@ -105,5 +108,6 @@
             <axis xyz = "0 0 1"/>
             <origin rpy="-${PId2} 0 ${PId2}"/>
-            <limit lower = "-${PI}" upper = "${PI}" effort = "50" velocity = "10"/>
+            <dynamics damping="0.7"/>
+            <limit lower = "-${PI}" upper = "${PI}" effort = "40" velocity = "1000"/>
         </joint>
         <joint name="link_3_to_link_4" type="revolute">
@@ -112,5 +116,6 @@
             <axis xyz = "0 0 1"/>
             <origin rpy="-${PId2} 0 -${PId2}" xyz = "0 0 0.27597"/>
-            <limit lower = "-${PI}" upper = "${PI}" effort = "50" velocity = "10"/>
+            <dynamics damping="0.7"/>
+            <limit lower = "-${PI}" upper = "${PI}" effort = "40" velocity = "1000"/>
         </joint>
         <joint name="link_4_to_link_5" type="revolute">
@@ -119,6 +124,57 @@
             <axis xyz = "0 0 1"/>
             <origin rpy="${PId2} 0 ${PId2}"/>
-            <limit lower = "-${PI}" upper = "${PI}" effort = "50" velocity = "10"/>
+            <dynamics damping="0.7"/>
+            <limit lower = "-${PI}" upper = "${PI}" effort = "40" velocity = "1000"/>
         </joint>
+        <transmission name="tran1">
+            <type>transmission_interface/SimpleTransmission</type>
+            <joint name="arm_base_to_link_1">
+                <hardwareInterface>EffortJointInterface</hardwareInterface>
+            </joint>
+            <actuator name="motor1">
+                <hardwareInterface>EffortJointInterface</hardwareInterface>
+                <mechanicalReduction>1</mechanicalReduction>
+            </actuator>
+        </transmission>
+        <transmission name="tran2">
+            <type>transmission_interface/SimpleTransmission</type>
+            <joint name="link_1_to_link_2">
+                <hardwareInterface>EffortJointInterface</hardwareInterface>
+            </joint>
+            <actuator name="motor2">
+                <hardwareInterface>EffortJointInterface</hardwareInterface>
+                <mechanicalReduction>1</mechanicalReduction>
+            </actuator>
+        </transmission>
+        <transmission name="tran3">
+            <type>transmission_interface/SimpleTransmission</type>
+            <joint name="link_2_to_link_3">
+                <hardwareInterface>EffortJointInterface</hardwareInterface>
+            </joint>
+            <actuator name="motor3">
+                <hardwareInterface>EffortJointInterface</hardwareInterface>
+                <mechanicalReduction>1</mechanicalReduction>
+            </actuator>
+        </transmission>
+        <transmission name="tran4">
+            <type>transmission_interface/SimpleTransmission</type>
+            <joint name="link_3_to_link_4">
+                <hardwareInterface>EffortJointInterface</hardwareInterface>
+            </joint>
+            <actuator name="motor4">
+                <hardwareInterface>EffortJointInterface</hardwareInterface>
+                <mechanicalReduction>1</mechanicalReduction>
+            </actuator>
+        </transmission>
+        <transmission name="tran5">
+            <type>transmission_interface/SimpleTransmission</type>
+            <joint name="link_4_to_link_5">
+                <hardwareInterface>EffortJointInterface</hardwareInterface>
+            </joint>
+            <actuator name="motor5">
+                <hardwareInterface>EffortJointInterface</hardwareInterface>
+                <mechanicalReduction>1</mechanicalReduction>
+            </actuator>
+        </transmission>
     </xacro:macro>
 </robot>

File: kumara_description/urdf/kumara_properties.xacro (robot description, xacro)
@@ -4,4 +4,8 @@
 	<xacro:property name="PI" value="3.1415926535897931"/>
 	<xacro:property name="PId2" value="1.57079632679"/>
+	<!-- BASE -->
+	<xacro:property name="BASE_WIDTH" value="0.5"/>
+	<xacro:property name="BASE_LENGTH" value="0.634"/>
+	<xacro:property name="BASE_HEIGHT" value="0.23"/>
 	<!-- ARM -->
 	<xacro:property name="L1" value="0.13764"/>
