Commit message: add base planar joint and base contorl

File: kumara_description/urdf/kumara.xacro (robot description, xacro)
@@ -9,6 +9,11 @@
     <xacro:include filename="$(find kumara_description)/urdf/kumara_base.gazebo" />
     <!-- ARM -->
-    <xacro:include filename="$(find kumara_description)/urdf/kumara_arm.xacro" />
+    <xacro:include filename="$(find kumara_description)/urdf/kumara_arm.xacro" />\
+    <!-- UTILITIES -->
+    <xacro:include filename="$(find kumara_description)/urdf/planar_joint.xacro" />
+    <!-- COMPONENTS -->
     <xacro:kumaraRA parent = "chassis"/>
+    <xacro:planar_joint prefix = "base" parent = "world" child = "base_footprint"/>
+    <link name="world"/>
     <link name="base_footprint"/>
     <link name="chassis">
@@ -30,10 +35,8 @@
         </visual>
     </link>
-    <joint name="base_footprint_to_base_link" type="fixed">
+    <joint name="base_footprint_to_chassis" type="fixed">
         <parent link="base_footprint"/>
         <child link="chassis"/>
         <origin xyz="0 0 ${BASE_HEIGHT}"/>
-        <axis xyz = "0 1 0"/>
-        <limit effort = "50" velocity = "10"/>
     </joint>
 </robot>

Commit message: add neck and head

File: kumara_description/urdf/kumara.xacro (robot description, xacro)
@@ -9,5 +9,7 @@
     <xacro:include filename="$(find kumara_description)/urdf/kumara_base.gazebo" />
     <!-- ARM -->
-    <xacro:include filename="$(find kumara_description)/urdf/kumara_arm.xacro" />\
+    <xacro:include filename="$(find kumara_description)/urdf/kumara_arm.xacro" />
+    <!-- NECK -->
+    <xacro:include filename="$(find kumara_description)/urdf/kumara_neck.xacro" />
     <!-- UTILITIES -->
     <xacro:include filename="$(find kumara_description)/urdf/planar_joint.xacro" />
@@ -15,4 +17,5 @@
     <xacro:kumaraRA parent = "chassis"/>
     <xacro:planar_joint prefix = "base" parent = "world" child = "base_footprint"/>
+    <xacro:kumara_neck parent = "chassis" child = "head_link"/>
     <link name="world"/>
     <link name="base_footprint"/>
@@ -40,3 +43,21 @@
         <origin xyz="0 0 ${BASE_HEIGHT}"/>
     </joint>
+    <link name="head_link">
+        <collision>
+			<origin xyz="0 0 -${0.23/2}"/>
+			<geometry>
+				<box size = "0.1 0.1 0.1"/>
+			</geometry>
+		</collision>
+		<inertial>
+            <origin xyz="0 0 0"/>
+			<mass value = "1"/>
+			<inertia ixx = "0.89" iyy = "1.1" izz = "1.64" ixy = "0" ixz = "0" iyz = "0"/>
+		</inertial>
+        <visual>
+            <geometry>
+                <mesh filename="package://kumara_description/meshes/head/head.STL" scale="1 1 1"/>
+            </geometry>
+        </visual>
+    </link>
 </robot>

File: kumara_description/urdf/kumara_arm.xacro (robot description, xacro)
@@ -130,8 +130,8 @@
             <type>transmission_interface/SimpleTransmission</type>
             <joint name="arm_base_to_link_1">
-                <hardwareInterface>EffortJointInterface</hardwareInterface>
+                <hardwareInterface>hardware_interface/EffortJointInterface</hardwareInterface>
             </joint>
             <actuator name="motor1">
-                <hardwareInterface>EffortJointInterface</hardwareInterface>
+                <hardwareInterface>hardware_interface/EffortJointInterface</hardwareInterface>
                 <mechanicalReduction>1</mechanicalReduction>
             </actuator>
@@ -140,8 +140,8 @@
             <type>transmission_interface/SimpleTransmission</type>
             <joint name="link_1_to_link_2">
-                <hardwareInterface>EffortJointInterface</hardwareInterface>
+                <hardwareInterface>hardware_interface/EffortJointInterface</hardwareInterface>
             </joint>
             <actuator name="motor2">
-                <hardwareInterface>EffortJointInterface</hardwareInterface>
+                <hardwareInterface>hardware_interface/EffortJointInterface</hardwareInterface>
                 <mechanicalReduction>1</mechanicalReduction>
             </actuator>
@@ -150,8 +150,8 @@
             <type>transmission_interface/SimpleTransmission</type>
             <joint name="link_2_to_link_3">
-                <hardwareInterface>EffortJointInterface</hardwareInterface>
+                <hardwareInterface>hardware_interface/EffortJointInterface</hardwareInterface>
             </joint>
             <actuator name="motor3">
-                <hardwareInterface>EffortJointInterface</hardwareInterface>
+                <hardwareInterface>hardware_interface/EffortJointInterface</hardwareInterface>
                 <mechanicalReduction>1</mechanicalReduction>
             </actuator>
@@ -160,8 +160,8 @@
             <type>transmission_interface/SimpleTransmission</type>
             <joint name="link_3_to_link_4">
-                <hardwareInterface>EffortJointInterface</hardwareInterface>
+                <hardwareInterface>hardware_interface/EffortJointInterface</hardwareInterface>
             </joint>
             <actuator name="motor4">
-                <hardwareInterface>EffortJointInterface</hardwareInterface>
+                <hardwareInterface>hardware_interface/EffortJointInterface</hardwareInterface>
                 <mechanicalReduction>1</mechanicalReduction>
             </actuator>
@@ -170,8 +170,8 @@
             <type>transmission_interface/SimpleTransmission</type>
             <joint name="link_4_to_link_5">
-                <hardwareInterface>EffortJointInterface</hardwareInterface>
+                <hardwareInterface>hardware_interface/EffortJointInterface</hardwareInterface>
             </joint>
             <actuator name="motor5">
-                <hardwareInterface>EffortJointInterface</hardwareInterface>
+                <hardwareInterface>hardware_interface/EffortJointInterface</hardwareInterface>
                 <mechanicalReduction>1</mechanicalReduction>
             </actuator>

File: kumara_description/urdf/planar_joint.xacro (robot description, xacro)
@@ -55,8 +55,8 @@
             <type>transmission_interface/SimpleTransmission</type>
             <joint name="${prefix}_x_axis_joint">
-                <hardwareInterface>EffortJointInterface</hardwareInterface>
+                <hardwareInterface>hardware_interface/EffortJointInterface</hardwareInterface>
             </joint>
             <actuator name="${prefix}_x_prismatic">
-                <hardwareInterface>EffortJointInterface</hardwareInterface>
+                <hardwareInterface>hardware_interface/EffortJointInterface</hardwareInterface>
                 <mechanicalReduction>1</mechanicalReduction>
             </actuator>
@@ -65,8 +65,8 @@
             <type>transmission_interface/SimpleTransmission</type>
             <joint name="${prefix}_y_axis_joint">
-                <hardwareInterface>EffortJointInterface</hardwareInterface>
+                <hardwareInterface>hardware_interface/EffortJointInterface</hardwareInterface>
             </joint>
             <actuator name="${prefix}_y_prismatic">
-                <hardwareInterface>EffortJointInterface</hardwareInterface>
+                <hardwareInterface>hardware_interface/EffortJointInterface</hardwareInterface>
                 <mechanicalReduction>1</mechanicalReduction>
             </actuator>
@@ -75,8 +75,8 @@
             <type>transmission_interface/SimpleTransmission</type>
             <joint name="${prefix}_z_axis_joint">
-                <hardwareInterface>EffortJointInterface</hardwareInterface>
+                <hardwareInterface>hardware_interface/EffortJointInterface</hardwareInterface>
             </joint>
             <actuator name="${prefix}_z_revolute">
-                <hardwareInterface>EffortJointInterface</hardwareInterface>
+                <hardwareInterface>hardware_interface/EffortJointInterface</hardwareInterface>
                 <mechanicalReduction>1</mechanicalReduction>
             </actuator>

Commit message: Add some document and Gazebo world environment

File: kumara_description/urdf/kumara.xacro (robot description, xacro)
@@ -5,4 +5,7 @@
             <robotNamespace>/kumara</robotNamespace>
         </plugin>
+        <!-- <plugin name="gazebo_cosim" filename="~/GazeboPlugin/export/lib/libGazeboCoSimPlugin.so">
+            <portNumber>14581</portNumber>
+        </plugin> -->
     </gazebo>
     <xacro:include filename="$(find kumara_description)/urdf/kumara_properties.xacro" />
@@ -20,5 +23,5 @@
     <xacro:planar_joint prefix = "base" parent = "world" child = "base_footprint"/>
     <xacro:kumara_neck parent = "chassis" child = "head_link"/>
-    <xacro:kumara_camera parent = "head_link"/>
+    <xacro:kumara_camera parent = "head_link" offset_from_parent = "0.072 0 0.1257"/>
     <link name="world"/>
     <link name="base_footprint"/>
@@ -64,3 +67,6 @@
         </visual>
     </link>
+    <gazebo reference="head_link">
+		<material>Gazebo/Grey</material>
+	</gazebo>
 </robot>

File: kumara_description/urdf/kumara_camera.xacro (robot description, xacro)
@@ -2,8 +2,7 @@
 <robot name="KumaraCamera" xmlns:xacro="http://www.ros.org/wiki/xacro">
     <xacro:include filename="$(find kumara_description)/urdf/kumara_properties.xacro" />
-    <xacro:macro name="kumara_camera" params="parent">
+    <xacro:macro name="kumara_camera" params="parent offset_from_parent">
         <joint name="camera_joint" type="fixed">
-            <axis xyz="0 1 0" />
-            <origin xyz="0.1 0 0.15" rpy="0 0 0"/>
+            <origin xyz="${offset_from_parent}" rpy="0 0 0"/>
             <parent link="${parent}"/>
             <child link="camera_link"/>
@@ -12,43 +11,45 @@
         <link name="camera_link">
             <collision>
-            <origin xyz="0 0 0" rpy="0 0 0"/>
-            <geometry>
-            <box size="0.01 0.01 0.01"/>
-            </geometry>
+                <origin xyz="0 0 0" rpy="0 0 0"/>
+                <geometry>
+                    <box size="0.01 0.01 0.01"/>
+                </geometry>
             </collision>
             <visual>
-            <origin xyz="0 0 0" rpy="0 0 0"/>
-            <geometry>
-            <box size="0.01 0.01 0.01"/>
-            </geometry>
-            <material name="red"/>
+                <origin xyz="0 0 0" rpy="0 0 0"/>
+                <geometry>
+                    <mesh filename="package://kumara_description/meshes/zedmini_camera.STL" scale="1 1 1"/>
+                </geometry>
+                <material name="red"/>
             </visual>
             <inertial>
-            <mass value="1e-5" />
-            <origin xyz="0 0 0" rpy="0 0 0"/>
-            <inertia ixx="1e-6" ixy="0" ixz="0" iyy="1e-6" iyz="0" izz="1e-6" />
+                <mass value="1e-5" />
+                <origin xyz="0 0 0" rpy="0 0 0"/>
+                <inertia ixx="1e-6" ixy="0" ixz="0" iyy="1e-6" iyz="0" izz="1e-6" />
             </inertial>
         </link>
         <gazebo reference="camera_link">
+            <material>Gazebo/Black</material>
             <sensor type="camera" name="camera1">
-            <update_rate>30.0</update_rate>
+            <update_rate>60.0</update_rate>
             <camera name="head">
-                <horizontal_fov>1.3962634</horizontal_fov>
+                <vertical_fov>1.0472</vertical_fov>
+                <horizontal_fov>1.5708</horizontal_fov>
                 <image>
-                <width>800</width>
-                <height>800</height>
-                <format>R8G8B8</format>
+                    <width>2560</width>
+                    <height>720</height>
+                    <format>R8G8B8</format>
                 </image>
                 <clip>
-                <near>0.02</near>
-                <far>300</far>
+                    <near>0.035</near>
+                    <far>300</far>
                 </clip>
                 <noise>
-                <type>gaussian</type>
-                <!-- Noise is sampled independently per pixel on each frame.
-                    That pixel's noise value is added to each of its color
-                    channels, which at that point lie in the range [0,1]. -->
-                <mean>0.0</mean>
-                <stddev>0.007</stddev>
+                    <type>gaussian</type>
+                    <!-- Noise is sampled independently per pixel on each frame.
+                        That pixel's noise value is added to each of its color
+                        channels, which at that point lie in the range [0,1]. -->
+                    <mean>0.0</mean>
+                    <stddev>0.007</stddev>
                 </noise>
             </camera>

Commit message: Add LIDAR

File: kumara_description/urdf/kumara.xacro (robot description, xacro)
@@ -16,5 +16,7 @@
     <xacro:include filename="$(find kumara_description)/urdf/kumara_neck.xacro" />
     <!-- CAMERA -->
-    <xacro:include filename="$(find kumara_description)/urdf/kumara_camera.xacro" />
+    <xacro:include filename="$(find kumara_description)/urdf/zed_mini.xacro" />
+    <!-- LIDAR -->
+    <xacro:include filename="$(find kumara_description)/urdf/rplidar_a2.xacro" />
     <!-- UTILITIES -->
     <xacro:include filename="$(find kumara_description)/urdf/planar_joint.xacro" />
@@ -23,5 +25,6 @@
     <xacro:planar_joint prefix = "base" parent = "world" child = "base_footprint"/>
     <xacro:kumara_neck parent = "chassis" child = "head_link"/>
-    <xacro:kumara_camera parent = "head_link" offset_from_parent = "0.072 0 0.1257"/>
+    <xacro:zed_mini parent = "head_link" offset_from_parent = "0.072 0 0.1257"/>
+    <xacro:rplidar_a2 suffix = "front" parent = "chassis" offset_from_parent = "-0.1 0 0.06"/>
     <link name="world"/>
     <link name="base_footprint"/>

File: kumara_description/urdf/zed_mini.xacro (robot description, xacro)
@@ -1,6 +1,6 @@
 <?xml version="1.0"?>
-<robot name="KumaraCamera" xmlns:xacro="http://www.ros.org/wiki/xacro">
+<robot name="zed_mini" xmlns:xacro="http://www.ros.org/wiki/xacro">
     <xacro:include filename="$(find kumara_description)/urdf/kumara_properties.xacro" />
-    <xacro:macro name="kumara_camera" params="parent offset_from_parent">
+    <xacro:macro name="zed_mini" params="parent offset_from_parent">
         <joint name="camera_joint" type="fixed">
             <origin xyz="${offset_from_parent}" rpy="0 0 0"/>
@@ -21,5 +21,4 @@
                     <mesh filename="package://kumara_description/meshes/zedmini_camera.STL" scale="1 1 1"/>
                 </geometry>
-                <material name="red"/>
             </visual>
             <inertial>

Commit message: Add message type in the documentation table and add ultrasonic sensor capability

File: kumara_description/urdf/kumara.xacro (robot description, xacro)
@@ -15,8 +15,8 @@
     <!-- NECK -->
     <xacro:include filename="$(find kumara_description)/urdf/kumara_neck.xacro" />
-    <!-- CAMERA -->
+    <!-- SENSORS -->
     <xacro:include filename="$(find kumara_description)/urdf/zed_mini.xacro" />
-    <!-- LIDAR -->
     <xacro:include filename="$(find kumara_description)/urdf/rplidar_a2.xacro" />
+    <xacro:include filename="$(find kumara_description)/urdf/sonar.xacro" />
     <!-- UTILITIES -->
     <xacro:include filename="$(find kumara_description)/urdf/planar_joint.xacro" />
@@ -26,5 +26,24 @@
     <xacro:kumara_neck parent = "chassis" child = "head_link"/>
     <xacro:zed_mini parent = "head_link" offset_from_parent = "0.072 0 0.1257"/>
-    <xacro:rplidar_a2 suffix = "front" parent = "chassis" offset_from_parent = "-0.1 0 0.06"/>
+    <xacro:rplidar_a2 prefix = "front"
+                parent = "chassis"
+                offset_from_parent = "-0.1 0 0.06"
+                visualize = "false"/>
+    <xacro:sonar prefix = "left"
+                parent = "chassis"
+                offset_from_parent = "0 0.24 -0.05"
+                rotate_from_parent = "0 0 ${PId2}"
+                max_range = "1.5"
+                min_range = "0.03"
+                fov = "0.12"
+                visualize = "true"/>
+    <xacro:sonar prefix = "right"
+                parent = "chassis"
+                offset_from_parent = "0 -0.24 -0.05"
+                rotate_from_parent = "0 0 -${PId2}"
+                max_range = "1.5"
+                min_range = "0.03"
+                fov = "0.12"
+                visualize = "true"/>
     <link name="world"/>
     <link name="base_footprint"/>

File: kumara_description/urdf/rplidar_a2.xacro (robot description, xacro)
@@ -2,11 +2,11 @@
 <robot name="rplidar_a2" xmlns:xacro="http://www.ros.org/wiki/xacro">
     <xacro:include filename="$(find kumara_description)/urdf/kumara_properties.xacro" />
-    <xacro:macro name="rplidar_a2" params="suffix parent offset_from_parent">
-        <joint name="rplidar_joint_${suffix}" type="fixed">
+    <xacro:macro name="rplidar_a2" params="prefix parent offset_from_parent visualize">
+        <joint name="${prefix}_rplidar_joint" type="fixed">
             <origin xyz="${offset_from_parent}" rpy="0 0 0"/>
             <parent link="${parent}"/>
-            <child link="rplidar_link_${suffix}"/>
+            <child link="${prefix}_rplidar_link"/>
         </joint>
-        <link name="rplidar_link_${suffix}">
+        <link name="${prefix}_rplidar_link">
             <visual>
                 <origin xyz="0 0 -0.03" rpy="0 0 0"/>
@@ -22,9 +22,9 @@
             </inertial>
         </link>
-        <gazebo reference="rplidar_link_${suffix}">
+        <gazebo reference="${prefix}_rplidar_link">
             <material>Gazebo/Grey</material>
-            <sensor type="ray" name="rplidar_a2_${suffix}">
+            <sensor type="ray" name="${prefix}_rplidar_a2">
                 <pose>0 0 0 0 0 0</pose>
-                <visualize>true</visualize>
+                <visualize>${visualize}</visualize>
                 <update_rate>10</update_rate>
                 <ray>
@@ -52,7 +52,7 @@
                     </noise>
                 </ray>
-                <plugin name="gazebo_ros_lidar_${suffix}" filename="libgazebo_ros_laser.so">
-                    <topicName>/kumara/laser_${suffix}/scan</topicName>
-                    <frameName>rplidar_link_${suffix}</frameName>
+                <plugin name="gazebo_ros_${prefix}_lidar" filename="libgazebo_ros_laser.so">
+                    <topicName>/kumara/${prefix}_laser/scan</topicName>
+                    <frameName>${prefix}_rplidar_link</frameName>
                 </plugin>
             </sensor>
