Commit message: Add sonar, and body  visual, and mount some sensors to the intended position

File: kumara_description/urdf/kumara.xacro (robot description, xacro)
@@ -10,5 +10,8 @@
     </gazebo>
     <xacro:include filename="$(find kumara_description)/urdf/kumara_properties.xacro" />
+    <!-- BASE -->
     <xacro:include filename="$(find kumara_description)/urdf/kumara_base.gazebo" />
+    <!-- <xacro:include filename="$(find kumara_description)/urdf/omni_steering.xacro" /> -->
+    <xacro:include filename="$(find kumara_description)/urdf/planar_joint.xacro" />
     <!-- ARM -->
     <xacro:include filename="$(find kumara_description)/urdf/kumara_arm.xacro" />
@@ -19,30 +22,61 @@
     <xacro:include filename="$(find kumara_description)/urdf/rplidar_a2.xacro" />
     <xacro:include filename="$(find kumara_description)/urdf/sonar.xacro" />
-    <!-- UTILITIES -->
-    <xacro:include filename="$(find kumara_description)/urdf/planar_joint.xacro" />
     <!-- COMPONENTS -->
     <xacro:kumaraRA parent = "chassis"/>
     <xacro:planar_joint prefix = "base" parent = "world" child = "base_footprint"/>
+    <!-- <xacro:omni_steering/> -->
     <xacro:kumara_neck parent = "chassis" child = "head_link"/>
     <xacro:zed_mini parent = "head_link" offset_from_parent = "0.072 0 0.1257"/>
     <xacro:rplidar_a2 prefix = "front"
                 parent = "chassis"
-                offset_from_parent = "-0.1 0 0.06"
+                offset_from_parent = "0.27 0 0.03"
                 visualize = "false"/>
     <xacro:sonar prefix = "left"
                 parent = "chassis"
-                offset_from_parent = "0 0.24 -0.05"
+                offset_from_parent = "0 0.25 -0.05025"
                 rotate_from_parent = "0 0 ${PId2}"
-                max_range = "1.5"
+                max_range = "4"
                 min_range = "0.03"
-                fov = "0.12"
+                fov = "0.08"
                 visualize = "true"/>
     <xacro:sonar prefix = "right"
                 parent = "chassis"
-                offset_from_parent = "0 -0.24 -0.05"
+                offset_from_parent = "0 -0.25 -0.05025"
                 rotate_from_parent = "0 0 -${PId2}"
-                max_range = "1.5"
+                max_range = "4"
                 min_range = "0.03"
-                fov = "0.12"
+                fov = "0.08"
+                visualize = "true"/>
+    <xacro:sonar prefix = "front_right"
+                parent = "chassis"
+                offset_from_parent = "0.317 -0.173 -0.02525"
+                rotate_from_parent = "0 0 0"
+                max_range = "4"
+                min_range = "0.03"
+                fov = "0.08"
+                visualize = "true"/>
+    <xacro:sonar prefix = "front_left"
+                parent = "chassis"
+                offset_from_parent = "0.317 0.173 -0.02525"
+                rotate_from_parent = "0 0 0"
+                max_range = "4"
+                min_range = "0.03"
+                fov = "0.08"
+                visualize = "true"/>
+    <xacro:sonar prefix = "back_right"
+                parent = "chassis"
+                offset_from_parent = "-0.317 -0.173 -0.02525"
+                rotate_from_parent = "0 0 ${PI}"
+                max_range = "4"
+                min_range = "0.03"
+                fov = "0.08"
+                visualize = "true"/>
+    <xacro:sonar prefix = "back_left"
+                parent = "chassis"
+                offset_from_parent = "-0.317 0.173 -0.02525"
+                rotate_from_parent = "0 0 ${PI}"
+                max_range = "4"
+                min_range = "0.03"
+                fov = "0.08"
                 visualize = "true"/>
     <link name="world"/>
@@ -66,8 +100,25 @@
         </visual>
     </link>
+    <link name="body_link">
+		<inertial>
+            <origin xyz="0 0 0"/>
+			<mass value = "28"/>
+			<inertia ixx = "0.89" iyy = "1.1" izz = "1.64" ixy = "0" ixz = "0" iyz = "0"/>
+		</inertial>
+        <visual>
+            <geometry>
+                <mesh filename="package://kumara_description/meshes/bodyPlaceHolderV1.STL" scale="1 1 1"/>
+            </geometry>
+        </visual>
+    </link>
     <joint name="base_footprint_to_chassis" type="fixed">
         <parent link="base_footprint"/>
         <child link="chassis"/>
         <origin xyz="0 0 ${BASE_HEIGHT}"/>
+    </joint>
+    <joint name="chassis_to_body_link" type="fixed">
+        <parent link="chassis"/>
+        <child link="body_link"/>
+        <origin xyz = "0.1795 0 0"/>
     </joint>
     <link name="head_link">
@@ -92,3 +143,6 @@
 		<material>Gazebo/Grey</material>
 	</gazebo>
+    <gazebo reference="body_link">
+		<material>Gazebo/Grey</material>
+	</gazebo>
 </robot>

File: kumara_description/urdf/planar_joint.xacro (robot description, xacro)
@@ -2,8 +2,10 @@
 <robot name="PlanarJoint" xmlns:xacro="http://www.ros.org/wiki/xacro">
     <xacro:macro name="planar_joint" params="prefix parent child">
+        <xacro:property name="LINEAR_DAMP" value="15"/>
+        <xacro:property name="ANGULAR_DAMP" value="8"/>
         <link name="${prefix}_x_axis_link">
             <inertial>
                 <origin rpy="0.0 0 0" xyz="0 0 0"/>
-                <mass value="0.01" />
+                <mass value="1e-5" />
                 <inertia ixx="0" ixy="0.0" ixz="0.0" iyy="0" iyz="0.0" izz="0"/>
             </inertial>
@@ -11,5 +13,5 @@
                 <origin rpy="0.0 0 0" xyz="0 0 0"/>
                 <geometry>
-                    <box size="0.000001 0.000001 0.000001"/>
+                    <box size="1e-6 1e-6 1e-6"/>
                 </geometry>
             </visual>
@@ -21,10 +23,10 @@
             <axis xyz="1 0 0" />
             <limit effort="10000" lower="-1000.0" upper="1000.0" velocity="1000" />
-            <dynamics damping="10.0" />
+            <dynamics damping="${LINEAR_DAMP}" />
         </joint>
         <link name="${prefix}_y_axis_link">
             <inertial>
                 <origin rpy="0.0 0 0" xyz="0 0 0"/>
-                <mass value="0.01" />
+                <mass value="1e-5" />
                 <inertia ixx="0" ixy="0.0" ixz="0.0" iyy="0" iyz="0.0" izz="0"/>
             </inertial>
@@ -32,5 +34,5 @@
                 <origin rpy="0.0 0 0" xyz="0 0 0"/>
                 <geometry>
-                    <box size="0.000001 0.000001 0.000001"/>
+                    <box size="1e-6 1e-6 1e-6"/>
                 </geometry>
             </visual>
@@ -42,5 +44,5 @@
             <axis xyz="0 1 0" />
             <limit effort="10000" lower="-1000.0" upper="1000.0" velocity="1000" />
-            <dynamics damping="10.0" />
+            <dynamics damping="${LINEAR_DAMP}" />
         </joint>
         <joint name="${prefix}_z_axis_joint" type="continuous">
@@ -50,5 +52,5 @@
             <axis xyz = "0 0 1"/>
             <limit effort = "10000" velocity = "1000"/>
-            <dynamics damping="10.0" />
+            <dynamics damping="${ANGULAR_DAMP}" />
         </joint>
         <transmission name="${prefix}_x_drive">

File: kumara_description/urdf/sonar.xacro (robot description, xacro)
@@ -12,6 +12,5 @@
                 <origin xyz="0 0 0" rpy="0 0 0"/>
                 <geometry>
-                    <!-- <mesh filename="package://kumara_description/meshes/sonar.STL" scale="1 1 1"/> -->
-                    <box size = "0.02 0.02 0.02"/>
+                    <mesh filename="package://kumara_description/meshes/ultrasonicSensor.STL" scale="1 1 1"/>
                 </geometry>
                 <material name="grey"/>

Commit message: The mass parameter of the head is now accurate

File: kumara_description/urdf/kumara.xacro (robot description, xacro)
@@ -124,13 +124,13 @@
     <link name="head_link">
         <collision>
-			<origin xyz="0 0 -${0.23/2}"/>
+			<origin xyz="0 0 0.07"/>
 			<geometry>
-				<box size = "0.1 0.1 0.1"/>
+				<box size = "0.1765 0.227 0.1562"/>
 			</geometry>
 		</collision>
 		<inertial>
-            <origin xyz="0 0 0"/>
-			<mass value = "1"/>
-			<inertia ixx = "0.89" iyy = "1.1" izz = "1.64" ixy = "0" ixz = "0" iyz = "0"/>
+            <origin xyz="0.03563 0.00117 0.02783"/>
+			<mass value = "1.3"/>
+			<inertia ixx="0.0058440886" iyy="0.0077612567" izz="0.006483092" ixy="-0.0000726954" ixz="0.00046124" iyz="0.00001826713"/>
 		</inertial>
         <visual>
