Commit message: Combine base's premitive joint action to single cmd_vel

File: kumara_description/urdf/kumara_neck.xacro (robot description, xacro)
@@ -21,5 +21,5 @@
             <child link="neck_tran_x" />
             <axis xyz="1 0 0" />
-            <limit effort="10000" lower="-0.2" upper="0.2" velocity="1000" />
+            <limit effort="10000" lower="-0.059" upper="0.059" velocity="1000" />
             <dynamics damping="2.0" />
         </joint>
@@ -42,5 +42,5 @@
             <child link="neck_tran_z" />
             <axis xyz="0 0 1" />
-            <limit effort="10000" lower="-0.2" upper="0.2" velocity="1000" />
+            <limit effort="10000" lower="-0.018" upper="0" velocity="1000" />
             <dynamics damping="2.0" />
         </joint>
@@ -63,5 +63,5 @@
             <child link="neck_rot_x" />
             <axis xyz="1 0 0" />
-            <limit effort="10000" lower="-${PI}" upper="${PI}" velocity="1000" />
+            <limit effort="10000" lower="-1.0472" upper="1.0472" velocity="1000" />
             <dynamics damping="2.0" />
         </joint>
@@ -84,5 +84,5 @@
             <child link="neck_rot_y" />
             <axis xyz="0 1 0" />
-            <limit effort="10000" lower="-${PI}" upper="${PI}" velocity="1000" />
+            <limit effort="10000" lower="-1.0472" upper="1.0472" velocity="1000" />
             <dynamics damping="2.0" />
         </joint>
