Commit message: updated the arm's visual but mass properties are not yet updated

File: kumara_description/urdf/kumara_arm.xacro (robot description, xacro)
@@ -9,9 +9,4 @@
                 <inertia ixx = "0.26" iyy = "0.26" izz = "0.01" ixy = "0" ixz = "0" iyz = "0"/>
             </inertial>
-            <visual>
-                <geometry>
-                    <mesh filename="package://kumara_description/meshes/arm/base_link.STL" scale="1 1 1"/>
-                </geometry>
-            </visual>
         </link>
         <link name="link_1">
@@ -56,10 +51,10 @@
         <link name="link_4">
             <inertial>
-                <origin rpy="${PId2} 0 ${PId2}"/>
+                <origin rpy="${PId2} 0 ${PId2}" xyz = "0 -${a1} 0"/>
                 <mass value = "1"/>
                 <inertia ixx = "0.26" iyy = "0.26" izz = "0.01" ixy = "0" ixz = "0" iyz = "0"/>
             </inertial>
             <visual>
-                <origin rpy="${PId2} 0 ${PId2}"/>
+                <origin rpy="${PId2} 0 ${PId2}" xyz = "0 -${a1} 0"/>
                 <geometry>
                     <mesh filename="package://kumara_description/meshes/arm/link_4.STL" scale="1 1 1"/>
@@ -99,5 +94,5 @@
             <child link="link_2"/>
             <axis xyz = "0 0 1"/>
-            <origin rpy="${PId2} 0 0" xyz = "0 0 0.13764"/>
+            <origin rpy="${PId2} 0 0" xyz = "0 0 ${L1}"/>
             <dynamics damping="0.7"/>
             <limit lower = "-${PI}" upper = "${PI}" effort = "40" velocity = "1000"/>
@@ -115,5 +110,5 @@
             <child link="link_4"/>
             <axis xyz = "0 0 1"/>
-            <origin rpy="-${PId2} 0 -${PId2}" xyz = "0 0 0.27597"/>
+            <origin rpy="-${PId2} 0 -${PId2}" xyz = "0 0 ${L2}"/>
             <dynamics damping="0.7"/>
             <limit lower = "-${PI}" upper = "${PI}" effort = "40" velocity = "1000"/>
@@ -123,5 +118,5 @@
             <child link="link_5"/>
             <axis xyz = "0 0 1"/>
-            <origin rpy="${PId2} 0 ${PId2}"/>
+            <origin rpy="${PId2} 0 ${PId2}" xyz = "0 -${a1} 0"/>
             <dynamics damping="0.7"/>
             <limit lower = "-${PI}" upper = "${PI}" effort = "40" velocity = "1000"/>

File: kumara_description/urdf/kumara_properties.xacro (robot description, xacro)
@@ -9,6 +9,7 @@
 	<xacro:property name="BASE_HEIGHT" value="0.23"/>
 	<!-- ARM -->
-	<xacro:property name="L1" value="0.13764"/>
-	<xacro:property name="L2" value="0.27597"/>
-	<xacro:property name="L3" value="0.14"/>
+	<xacro:property name="L1" value="0.168"/>
+	<xacro:property name="L2" value="0.269"/>
+	<xacro:property name="L3" value="0.173"/>
+	<xacro:property name="a1" value="0.02616"/>
 </robot>
